File: StrainGauge2.kicad_pcb (KiCad board)
At the start: 2 copper layers, 32.2 x 20.5 mm, 67 parts, among them P1 CONN_2, P2 CONN_2, P3 CONN_2, P4 CONN_1, P5 CONN_01X04, Q1 DMP21D5UFB4-7B, U1 TPS63001, U2 ADS1291/2, U3 NRF528XX-QFAA, U4 MPU-9250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

Commit message: Removed MPU from schematic and PCB.
Parts:
- removed C35, C36: 100nF, SM0402
- removed R11, R12: 10k, SM0402
- removed U4: MPU-9250, Housings_DFN_QFN:QFN-24_3x3mm_Pitch0.4mm
Routing:
- net DVDD: track 82.4 -> 70.3 mm, vias 11 -> 9
- net DGND: track 163.8 -> 152.2 mm
- net /IN2: track 10.5 -> 0.00 mm
- net /IN2-: track 8.42 -> 0.00 mm
- net /IN1: track 7.26 -> 0.00 mm
- net /SCL: track 6.40 -> 0.25 mm
- net /SDI: track 5.98 -> 0.00 mm
- net /IN1-: track 4.93 -> 0.00 mm
- net Net-(R1-Pad1): track 3.40 -> 0.00 mm
- net Net-(R3-Pad1): track 2.86 -> 0.00 mm
- net Net-(R4-Pad1): track 2.56 -> 0.00 mm
- net Net-(R2-Pad1): track 2.55 -> 0.00 mm
- net Net-(C35-Pad1): track 1.17 -> 0.00 mm

Commit message: Remove Bias Circuit from schematic and pcb. Finalized circuits with wheatstone bridges.
Parts:
- removed C4: 1.0nF-1.5nF, SM0402
- removed P4: CONN_1, Pin_Headers:Pin_Header_Straight_1x01_Pitch2.54mm
- added R11: 200k, SM0402, F.Cu at (293.1, 132.8)
- R1, R2, R3, R4: value 30k -> 200k
- R6: value 1MΩ -> 200k
- moved R6 5.43 mm to (293.3, 134.1), turned to 0 degrees
- moved P5 3.82 mm to (296.2, 130.8)
- moved R2 2.01 mm to (291.8, 138.2), turned to 270 degrees
- moved R4 0.71 mm to (291.9, 133.7), turned to 270 degrees
- moved R1 0.59 mm to (292.3, 136.7), turned to 180 degrees
- moved R3 0.50 mm to (292.3, 135.7), turned to 180 degrees
Connections:
- net /SCL renamed Net-(U3-Pad24)
- net /SDI renamed Net-(U3-Pad23)
- P5 pad 1: /IN2 -> DGND
- P5 pad 2: /IN2- -> /SG2_INPUT_1
- P5 pad 3: /IN1 -> /SG1_INPUT_1
- P5 pad 4: /IN1- -> DGND
- R1 pad 1: Net-(R1-Pad1) -> DVDD
- R1 pad 2: /IN1- -> /WB1_Vinverting
- R2 pad 1: Net-(R2-Pad1) -> /WB1_Vinverting
- R2 pad 2: /IN1 -> DGND
- R3 pad 1: Net-(R3-Pad1) -> DVDD
- R3 pad 2: /IN2- -> /SG1_INPUT_1
- R4 pad 1: Net-(R4-Pad1) -> DVDD
- R4 pad 2: /IN2 -> /WB2_Vinverting
- R6 pad 1: Net-(C4-Pad1) -> /WB2_Vinverting
- R6 pad 2: /BIASIN -> DGND
- U2 pad 28: Net-(C4-Pad1) -> Net-(U2-Pad28)
- U2 pad 29: /BIASIN -> Net-(U2-Pad29)
- U2 pad 3: Net-(R1-Pad1) -> /WB1_Vinverting
- U2 pad 30: /BIASIN -> Net-(U2-Pad30)
- U2 pad 4: Net-(R2-Pad1) -> /SG1_INPUT_1
- U2 pad 5: Net-(R3-Pad1) -> /WB2_Vinverting
- U2 pad 6: Net-(R4-Pad1) -> /SG2_INPUT_1
Routing:
- net DVDD: track 70.3 -> 86.2 mm, vias 9 -> 11
- net DGND: track 152.2 -> 165.7 mm, vias 11 -> 13
- net /BIASIN: track 11.1 -> 0.40 mm
- net /SG2_INPUT_1: track 0.00 -> 9.32 mm
- net /SG1_INPUT_1: track 0.00 -> 8.29 mm
- net Net-(C4-Pad1): track 7.23 -> 0.00 mm
- net /WB2_Vinverting: track 0.00 -> 4.72 mm
- net /WB1_Vinverting: track 0.00 -> 4.55 mm
Other:
- board text added: "2-Channel Strain Gauge Circuit"
- board text added: "nRF52-ADS1292 Strain Gauge - 04/26/19 Yeo Lab, GaTech"
- board text removed: "+"
- board text removed: "BIAS"
- board text removed: "MPU9250"
- board text removed: "nRF52-ADS1292-MPU ExG Prototype - 06/08/18 Yeo GaTech BNE Lab"
- board text removed: "—"
